Commit message: refactor:remove rizon urdf

File: flexiv_amr_description/fmr_300/urdf/FMR300.urdf (robot description, URDF)
Before this commit: robot FMR300, 21 links, 20 joints
Links:
- removed link AMR
- removed link flange
- removed link link1
- removed link link2
- removed link link3
- removed link link4
- removed link link5
- removed link link6
- removed link link7
- link base_link: mass 9.2 -> 250; geometry collision mesh filename=package://flexiv_amr_description/fmr_300/meshes/AMR.STL; visual mesh filename=package://flexiv_amr_description/fmr_300/meshes/AMR.STL
Joints:
- removed joint joint1
- removed joint joint2
- removed joint joint3
- removed joint joint4
- removed joint joint5
- removed joint joint6
- removed joint joint7
- removed joint link7_to_flange
- removed joint rizon10
- joint driving_wheel1: parent AMR -> base_link
- joint driving_wheel2: parent AMR -> base_link
- joint imu_joint: parent AMR -> base_link
- joint universal_wheel1: parent AMR -> base_link
- joint universal_wheel2: parent AMR -> base_link
- joint universal_wheel3: parent AMR -> base_link
- joint universal_wheel4: parent AMR -> base_link
